File: eagle/main/simple-spectro-pro.brd (EAGLE design)
At the start: 99.1 x 73.7 mm, 72 parts, among them IC1 MCP1703-33, IC2 MCP1703-50, IC3 MCP43X2ST, J1 RJ12RIGHTANGLE-RGB, J2 RJ12RIGHTANGLE-I2C, J3 RJ12RIGHTANGLE, Q1 DMP1045U, U1 MCP73831T, X2 8MHz, X3 1503_09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

Commit message: final version eagle v1.0.0
Parts:
- moved JP1 1.91 mm to (64.8, 67.3)
- moved CON_ISP1 1.91 mm to (7.62, 50.8)
- moved R6 1.27 mm to (7.62, 61.6)
Routing:
- net VCC: track 488.3 -> 497.6 mm
- net VBAT1: track 56.4 -> 59.9 mm
- net ISP+5V: track 154.9 -> 152.5 mm
- net MOSI: track 112.3 -> 110.4 mm
- net RESET: track 59.9 -> 58.0 mm
- net SCK: track 104.0 -> 102.5 mm
- net MISO: track 103.4 -> 102.1 mm
- net N$2: track 26.0 -> 24.8 mm
